File: Rochelle_circuit/Rochelle_circuit.kicad_sch (KiCad schematic)
At the start: 18 parts, among them U1 INA125, U2 LM358

Commit message: removed HP Filter
Parts:
- removed C2: 1.6u, symbol Device:C_Small
- removed R9: 1M, symbol Device:R_Small_US
- renumbered LiquidWire to LiquidWire1
Connections:
- net at R5.1: now also R7.1, U1.10 (Vo), U1.11 (Sense)
Other:
- note removed: "Cutoff Frequency at 0.1 Hz"
- note removed: "High-Pass filter"
- note removed: "Up until these points in the circuit, everything works."
